Commit message: Add build logs for hydroships_description package
- Created stderr.log and stdout.log to capture standard error and output during the build process.
- Added stdout_stderr.log to consolidate both stdout and stderr logs.
- Introduced streams.log to log the commands executed during the build.
- Generated logger_all.log for detailed debugging information during the build of hydroships_control and hydroships_description packages.

File: install/hydroships_description/share/hydroships_description/urdf/hydroships.urdf.xacro (robot description, xacro)
@@ -127,5 +127,7 @@
   <link name="camera_bottom_link"/>
   <joint name="camera_bottom_joint" type="fixed">
-    <origin xyz="0 0 ${-body_z/2}" rpy="0 1.5708 0"/>
+    <!-- Sedikit DI BAWAH sisi bawah mesh (z=-0.143) agar pandangan ke bawah tidak
+         terhalang badan ROV sendiri; port kamera bawah menghadap dasar kolam. -->
+    <origin xyz="0.02 0 -0.18" rpy="0 1.5708 0"/>
     <parent link="base_link"/>
     <child link="camera_bottom_link"/>
