Commit message: Buat ulang model visual ROV jadi primitif sederhana
Ganti mesh STL 12 MB (237k segitiga, hasil konversi FBX yang bentuknya
acak-acak & bikin rate kamera turun) dengan susunan primitif ringan
bergaya BlueROV Heavy: rangka kotak hitam + busa apung oranye + tabung
elektronik abu-abu + dome kamera depan (penanda haluan +X).

- Visual base_link kini box/cylinder, mengisi bbox desain 0.345x0.345x0.286 m
- Collision box (fisika/buoyancy) tidak diubah
- Sinkron salinan xacro di install/share
- Update PROBLEM.md: model visual RESOLVED tahap-1

Co-Authored-By: Claude Opus 4.8 <noreply@anthropic.com>
Claude-Session: https://claude.ai/code/session_01N4S9CvgPGGeAXaJ1PkDJat

File: install/hydroships_description/share/hydroships_description/urdf/hydroships.urdf.xacro (robot description, xacro)
@@ -18,7 +18,5 @@
   <xacro:property name="body_y" value="0.345"/>
   <xacro:property name="body_z" value="0.286"/>
-  <!-- Rotasi yaw mesh visual (rad) agar haluan/bow menghadap +X (arah surge).
-       Sesuaikan bila bow mesh menghadap arah lain: 1.5708=+90°, -1.5708=-90°, 3.14159=180°. -->
-  <xacro:property name="bow_yaw" value="0"/>
+  <!-- (bow_yaw dulu untuk memutar mesh; visual kini primitif dgn haluan tetap +X.) -->
   <!-- Massa base dipilih agar total near-neutral, sedikit positif buoyant. -->
   <xacro:property name="base_mass" value="33.6"/>
@@ -38,16 +36,51 @@
                izz="${izz}"/>
     </inertial>
-    <!-- Visual: mesh ROV asli (meshes/rov.stl, dari model/rov.fbx: node-transform
-         di-bake via PreTransformVertices lalu di-decimate; Fortress tak bisa FBX).
-         Mesh dalam MILIMETER (bbox 350.7 x 344.5 x 286 mm ≈ kotak desain) → scale 0.001.
-         Mesh sudah di-center di file, jadi origin xyz=0. rpy=0 0 ${bow_yaw}: arah bow
-         (+X) mungkin perlu diputar — lihat PROBLEM.md. Collision TETAP kotak (fisika). -->
-    <visual>
-      <origin xyz="0 0 0" rpy="0 0 ${bow_yaw}"/>
-      <geometry>
-        <mesh filename="package://hydroships_description/meshes/rov.stl" scale="0.001 0.001 0.001"/>
-      </geometry>
-      <material name="hydro_yellow">
-        <color rgba="0.9 0.75 0.1 1.0"/>
+    <!-- Visual: model SEDERHANA dari primitif (BUKAN mesh berat lagi).
+         Sebelumnya pakai meshes/rov.stl (12 MB, ~237k segitiga hasil konversi FBX)
+         yang bentuknya acak-acak & bikin rate kamera turun ~22→10 Hz (lihat PROBLEM.md).
+         Diganti susunan box/cylinder ringan bergaya BlueROV Heavy:
+           - rangka kotak HITAM (bagian bawah)
+           - busa apung ORANYE (bagian atas)
+           - tabung elektronik abu-abu + dome kamera depan (penanda haluan +X)
+         Total tetap mengisi bbox desain 0.345 x 0.345 x 0.286 m; bow = +X (arah surge).
+         Collision TETAP kotak (untuk fisika/buoyancy) — tak diubah. -->
+    <!-- Rangka utama (hitam) — bagian bawah badan. -->
+    <visual>
+      <origin xyz="0 0 -0.0465" rpy="0 0 0"/>
+      <geometry>
+        <box size="0.345 0.345 0.193"/>
+      </geometry>
+      <material name="hydro_frame_black">
+        <color rgba="0.10 0.10 0.11 1.0"/>
+      </material>
+    </visual>
+    <!-- Busa apung (oranye) — blok di atas, sedikit inset dari rangka. -->
+    <visual>
+      <origin xyz="0 0 0.0965" rpy="0 0 0"/>
+      <geometry>
+        <box size="0.315 0.335 0.093"/>
+      </geometry>
+      <material name="hydro_orange">
+        <color rgba="0.95 0.45 0.05 1.0"/>
+      </material>
+    </visual>
+    <!-- Tabung elektronik (abu-abu) — silinder membujur sumbu X di tengah badan. -->
+    <visual>
+      <origin xyz="0.0 0 0.005" rpy="0 1.5708 0"/>
+      <geometry>
+        <cylinder radius="0.058" length="0.30"/>
+      </geometry>
+      <material name="hydro_grey">
+        <color rgba="0.55 0.55 0.58 1.0"/>
+      </material>
+    </visual>
+    <!-- Dome kamera depan (abu gelap) — penanda haluan (+X). -->
+    <visual>
+      <origin xyz="0.175 0 0.005" rpy="0 1.5708 0"/>
+      <geometry>
+        <cylinder radius="0.045" length="0.02"/>
+      </geometry>
+      <material name="hydro_dome">
+        <color rgba="0.15 0.15 0.18 1.0"/>
       </material>
     </visual>
@@ -66,5 +99,5 @@
     axis  : arah dorong (unit vector) di frame body; juga sumbu putar propeller
   -->
-  <xacro:macro name="thruster" params="name xyz axis">
+  <xacro:macro name="thruster" params="name xyz axis visual_rpy='0 0 0' visual_offset='0 0 0'">
     <link name="${name}">
       <inertial>
@@ -75,10 +108,19 @@
       </inertial>
       <visual>
-        <origin xyz="0 0 0" rpy="0 0 0"/>
+        <origin xyz="${visual_offset}" rpy="${visual_rpy}"/>
         <geometry>
-          <cylinder radius="0.02" length="0.06"/>
+          <cylinder radius="0.012" length="0.05"/>
         </geometry>
         <material name="hydro_dark">
           <color rgba="0.1 0.1 0.12 1.0"/>
+        </material>
+      </visual>
+      <visual>
+        <origin xyz="${visual_offset}" rpy="${visual_rpy}"/>
+        <geometry>
+          <cylinder radius="0.024" length="0.008"/>
+        </geometry>
+        <material name="hydro_yellow">
+          <color rgba="0.9 0.75 0.1 1.0"/>
         </material>
       </visual>
@@ -95,15 +137,18 @@
     </joint>
   </xacro:macro>
-  <!-- ==================== 3 thruster horizontal ==================== -->
-  <!-- Susunan tangensial 120 deg (rh = 0.16 m). Mengontrol surge/sway/yaw.
-       phi = 90, 210, 330 deg; arah dorong d = (-sin phi, cos phi, 0). -->
-  <xacro:thruster name="thruster_1" xyz="0.0     0.16   0.0"  axis="-1.0  0.0   0.0"/>
-  <xacro:thruster name="thruster_2" xyz="-0.1386 -0.08  0.0"  axis="0.5  -0.866 0.0"/>
-  <xacro:thruster name="thruster_3" xyz="0.1386  -0.08  0.0"  axis="0.5   0.866 0.0"/>
-  <!-- ==================== 3 thruster vertikal ==================== -->
-  <!-- Arah dorong +z. Mengontrol heave/roll/pitch. -->
-  <xacro:thruster name="thruster_4" xyz="0.12   0.0    0.0"  axis="0.0  0.0  1.0"/>
-  <xacro:thruster name="thruster_5" xyz="-0.10  0.12   0.0"  axis="0.0  0.0  1.0"/>
-  <xacro:thruster name="thruster_6" xyz="-0.10 -0.12   0.0"  axis="0.0  0.0  1.0"/>
+    <!-- ==================== Thruster positions (diperbarui dari thruster_positions.csv) -->
+    <!-- Mapping sesuai klarifikasi pengguna:
+         thruster_1 = T200-E (vertikal)
+         thruster_2 = T200-F (vertikal)
+         thruster_3 = T100-C (depan horizontal)
+         thruster_4 = T100-A (depan horizontal)
+         thruster_5 = T100-B (lateral bawah horizontal)
+         thruster_6 = T100-D (belakang sentral vertikal) -->
+    <xacro:thruster name="thruster_1" xyz="0.1234 0.0275 0.0142" axis="0.0 0.0 1.0" visual_rpy="0 1.5708 0" visual_offset="0.008 0.004 0.000"/>
+    <xacro:thruster name="thruster_2" xyz="-0.1228 0.0290 0.0148" axis="0.0 0.0 1.0" visual_rpy="0 1.5708 0" visual_offset="0.008 -0.004 0.000"/>
+    <xacro:thruster name="thruster_3" xyz="0.1371 -0.1298 0.0336" axis="1.0 0.0 0.0" visual_rpy="1.5708 0 0" visual_offset="0.008 -0.002 -0.002"/>
+    <xacro:thruster name="thruster_4" xyz="-0.1371 -0.1296 0.0374" axis="1.0 0.0 0.0" visual_rpy="1.5708 0 0" visual_offset="0.008 0.002 -0.002"/>
+    <xacro:thruster name="thruster_5" xyz="0.0003 0.0455 -0.0994" axis="0.0 1.0 0.0" visual_rpy="0 0 1.5708" visual_offset="0.000 0.000 0.008"/>
+    <xacro:thruster name="thruster_6" xyz="-0.0003 0.1364 0.0403" axis="0.0 0.0 1.0" visual_rpy="0 1.5708 0" visual_offset="0.006 0.000 -0.001"/>
   <!-- ==================== Frame sensor (placeholder M3) ==================== -->
   <link name="imu_link"/>

File: src/hydroships_description/urdf/hydroships.urdf.xacro (robot description, xacro)
@@ -18,7 +18,5 @@
   <xacro:property name="body_y" value="0.345"/>
   <xacro:property name="body_z" value="0.286"/>
-  <!-- Rotasi yaw mesh visual (rad) agar haluan/bow menghadap +X (arah surge).
-       Sesuaikan bila bow mesh menghadap arah lain: 1.5708=+90°, -1.5708=-90°, 3.14159=180°. -->
-  <xacro:property name="bow_yaw" value="0"/>
+  <!-- (bow_yaw dulu untuk memutar mesh; visual kini primitif dgn haluan tetap +X.) -->
   <!-- Massa base dipilih agar total near-neutral, sedikit positif buoyant. -->
   <xacro:property name="base_mass" value="33.6"/>
@@ -38,16 +36,51 @@
                izz="${izz}"/>
     </inertial>
-    <!-- Visual: mesh ROV asli (meshes/rov.stl, dari model/rov.fbx: node-transform
-         di-bake via PreTransformVertices lalu di-decimate; Fortress tak bisa FBX).
-         Mesh dalam MILIMETER (bbox 350.7 x 344.5 x 286 mm ≈ kotak desain) → scale 0.001.
-         Mesh sudah di-center di file, jadi origin xyz=0. rpy=0 0 ${bow_yaw}: arah bow
-         (+X) mungkin perlu diputar — lihat PROBLEM.md. Collision TETAP kotak (fisika). -->
-    <visual>
-      <origin xyz="0 0 0" rpy="0 0 ${bow_yaw}"/>
-      <geometry>
-        <mesh filename="package://hydroships_description/meshes/rov.stl" scale="0.001 0.001 0.001"/>
-      </geometry>
-      <material name="hydro_yellow">
-        <color rgba="0.9 0.75 0.1 1.0"/>
+    <!-- Visual: model SEDERHANA dari primitif (BUKAN mesh berat lagi).
+         Sebelumnya pakai meshes/rov.stl (12 MB, ~237k segitiga hasil konversi FBX)
+         yang bentuknya acak-acak & bikin rate kamera turun ~22→10 Hz (lihat PROBLEM.md).
+         Diganti susunan box/cylinder ringan bergaya BlueROV Heavy:
+           - rangka kotak HITAM (bagian bawah)
+           - busa apung ORANYE (bagian atas)
+           - tabung elektronik abu-abu + dome kamera depan (penanda haluan +X)
+         Total tetap mengisi bbox desain 0.345 x 0.345 x 0.286 m; bow = +X (arah surge).
+         Collision TETAP kotak (untuk fisika/buoyancy) — tak diubah. -->
+    <!-- Rangka utama (hitam) — bagian bawah badan. -->
+    <visual>
+      <origin xyz="0 0 -0.0465" rpy="0 0 0"/>
+      <geometry>
+        <box size="0.345 0.345 0.193"/>
+      </geometry>
+      <material name="hydro_frame_black">
+        <color rgba="0.10 0.10 0.11 1.0"/>
+      </material>
+    </visual>
+    <!-- Busa apung (oranye) — blok di atas, sedikit inset dari rangka. -->
+    <visual>
+      <origin xyz="0 0 0.0965" rpy="0 0 0"/>
+      <geometry>
+        <box size="0.315 0.335 0.093"/>
+      </geometry>
+      <material name="hydro_orange">
+        <color rgba="0.95 0.45 0.05 1.0"/>
+      </material>
+    </visual>
+    <!-- Tabung elektronik (abu-abu) — silinder membujur sumbu X di tengah badan. -->
+    <visual>
+      <origin xyz="0.0 0 0.005" rpy="0 1.5708 0"/>
+      <geometry>
+        <cylinder radius="0.058" length="0.30"/>
+      </geometry>
+      <material name="hydro_grey">
+        <color rgba="0.55 0.55 0.58 1.0"/>
+      </material>
+    </visual>
+    <!-- Dome kamera depan (abu gelap) — penanda haluan (+X). -->
+    <visual>
+      <origin xyz="0.175 0 0.005" rpy="0 1.5708 0"/>
+      <geometry>
+        <cylinder radius="0.045" length="0.02"/>
+      </geometry>
+      <material name="hydro_dome">
+        <color rgba="0.15 0.15 0.18 1.0"/>
       </material>
     </visual>
