Commit message: fix: passive CoB offset + active pitch/roll-hold to stop ROV pitch drift
ROV was pitching nose-up indefinitely because CoG and CoB were coincident
(no passive restoring moment) and the stabilizer only closed loops on
depth/heading, leaving pitch/roll fully open-loop against a small residual
heave-allocation moment.

- Shift base_link collision origin (buoyancy source) up by cob.z so CoB
  sits above CoG, giving positive metacentric height for passive stability.
- Add pitch-hold and roll-hold PID loops in stabilizer.py as an active
  robustness layer, mirroring the existing heading-hold pattern.

Co-Authored-By: Claude Sonnet 5 <noreply@anthropic.com>

File: src/hydroships_description/urdf/hydroships.urdf.xacro (robot description, xacro)
@@ -102,7 +102,10 @@
       </material>
     </visual>
-    <!-- Collision box dipakai plugin Buoyancy untuk menghitung volume perpindahan. -->
+    <!-- Collision box dipakai plugin Buoyancy untuk menghitung volume perpindahan.
+         Origin digeser ke atas sebesar cob.z (relatif thd inertial origin/CoG di atas)
+         agar CoB (centroid box ini) berada di atas CoG -> metacentric height positif,
+         restoring moment pasif utk pitch/roll (lihat rov_params.yaml: cob). -->
     <collision>
-      <origin xyz="0 0 0" rpy="0 0 0"/>
+      <origin xyz="${rp['cob']['x']} ${rp['cob']['y']} ${rp['cob']['z']}" rpy="0 0 0"/>
       <geometry>
         <box size="${body_x} ${body_y} ${body_z}"/>

Commit message: fix(description): gripper tidak lagi menyumbang volume apung
Plugin gz Buoyancy menurunkan volume perpindahan air dari geometri
<collision>. Ketiga link gripper (gripper_base + dua jari) punya collision
box, sehingga ikut menghasilkan gaya apung yang tidak pernah masuk neraca
di rov_params.yaml -- neraca itu hanya menghitung box base_link.

Akibatnya (diukur dari SDF yang benar-benar di-spawn):

  volume terpindah  0.009406 m^3  (bukan 0.008729)
  net apung         +6.92 N       (bukan +0.28 N, 24.7x)
  CoB               +13.6 mm ke haluan
  momen trim        1.036 N*m bow-up vs pemulih maks 1.691 N*m
  trim pasif        tan(theta) = 0.0112/0.0183 -> 31.5 deg bow-up

ROV karena itu mengambang miring, dan dorongan "vertikal" terproyeksi jadi
gerak horizontal: pada uji open-loop, perintah heave menghasilkan simpangan
lateral 2.5 m tapi perpindahan vertikal <= 0.4 m. Ini yang sebelumnya
terbaca seolah-olah aktuator hanya menyalurkan ~10% gaya (P0-1a) -- salah
tafsir yang kini digantikan.

Contact fisik gripper tidak dibutuhkan: grasp memakai DetachableJoint +
proximity visual (gripper_logic.is_safe membaca offset QR, bukan kontak),
HANG di-skor dari odometri, dan kedua jari didokumentasikan sebagai
kosmetik. Jadi collision-nya dihapus, mengikuti idiom yang sudah dipakai
thruster di file yang sama.

Setelah perubahan ini (prediksi -> terukur runtime):

  volume terpindah  0.008729 m^3
  net apung         +0.28 N        (laju naik bebas 0.029 m/s vs prediksi 0.035)
  CoB               (0, 0, 20) mm
  trim pasif        prediksi 6.9 deg bow-down -> terukur +4.44 / +3.58 deg
                    (sebelumnya -29.6 / -44.1 deg)

Sisa ~7 deg berasal dari CoG sistem 2.37 mm di depan CoB; ditangani terpisah
di commit berikutnya supaya efek tiap perubahan terukur sendiri.

Co-Authored-By: Claude Opus 5 <noreply@anthropic.com>

File: src/hydroships_description/urdf/hydroships.urdf.xacro (robot description, xacro)
@@ -272,8 +272,12 @@
       <material name="hydro_grip"><color rgba="0.85 0.7 0.1 1.0"/></material>
     </visual>
-    <collision>
-      <origin xyz="0 0 0" rpy="0 0 0"/>
-      <geometry><box size="0.10 0.10 0.06"/></geometry>
-    </collision>
+    <!-- Tanpa collision: gripper tidak menambah volume apung (sama alasannya
+         dgn thruster di atas). Plugin Buoyancy menghitung volume perpindahan
+         dari geometri <collision>, jadi kotak collision di sini ikut jadi gaya
+         apung 5.9 N di x=+0.18 m — di luar neraca apung rov_params.yaml, dan
+         menggeser CoB ke haluan sehingga ROV trim bow-up ~31°. Contact fisik
+         tak dibutuhkan: grasp memakai DetachableJoint + proximity visual
+         (gripper_logic.is_safe), HANG di-skor dari odometri, dan kedua jari
+         kosmetik. Lihat docs/CHANGELOG.md. -->
   </link>
   <joint name="gripper_base_joint" type="fixed">
@@ -309,8 +313,6 @@
         <material name="hydro_jaw"><color rgba="0.95 0.8 0.2 1.0"/></material>
       </visual>
-      <collision>
-        <origin xyz="0.04 0 0" rpy="0 0 0"/>
-        <geometry><box size="0.08 0.016 0.03"/></geometry>
-      </collision>
+      <!-- Tanpa collision: jari kosmetik, tidak menjepit secara fisik dan tidak
+           boleh menambah volume apung (lihat catatan di gripper_base). -->
     </link>
     <joint name="gripper_${side}_joint" type="revolute">
