Commit message: Create Problem for NOTE

File: src/hydroships_description/urdf/hydroships.urdf.xacro (robot description, xacro)
@@ -163,4 +163,71 @@
     </sensor>
   </gazebo>
+  <!-- ==================== Gripper 2-DOF (Milestone 5) ==================== -->
+  <!-- Dua jari (kiri/kanan) berputar di sumbu z untuk membuka/menutup di bidang xy.
+       Dikontrol per-jari oleh gz JointPositionController (topic gz.msgs.Double, rad).
+       Node gripper_controller memetakan perintah "open"/"close" -> setpoint 2 jari. -->
+  <xacro:property name="grip_mass" value="0.03"/>
+  <link name="gripper_base_link">
+    <inertial>
+      <mass value="${grip_mass}"/>
+      <inertia ixx="1e-5" ixy="0" ixz="0" iyy="1e-5" iyz="0" izz="1e-5"/>
+    </inertial>
+    <visual>
+      <geometry><box size="0.05 0.10 0.04"/></geometry>
+      <material name="grip_dark"><color rgba="0.12 0.12 0.14 1.0"/></material>
+    </visual>
+    <collision><geometry><box size="0.05 0.10 0.04"/></geometry></collision>
+  </link>
+  <joint name="gripper_base_joint" type="fixed">
+    <origin xyz="0.20 0 -0.10" rpy="0 0 0"/>
+    <parent link="base_link"/>
+    <child link="gripper_base_link"/>
+  </joint>
+  <!-- Macro satu jari: reflect = +1 (kiri, +y) / -1 (kanan, -y). -->
+  <xacro:macro name="finger" params="name reflect">
+    <link name="${name}_link">
+      <inertial>
+        <origin xyz="0.045 0 0" rpy="0 0 0"/>
+        <mass value="0.01"/>
+        <inertia ixx="1e-6" ixy="0" ixz="0" iyy="1e-6" iyz="0" izz="1e-6"/>
+      </inertial>
+      <visual>
+        <origin xyz="0.045 0 0" rpy="0 0 0"/>
+        <geometry><box size="0.09 0.018 0.03"/></geometry>
+        <material name="grip_yellow"><color rgba="0.9 0.75 0.1 1.0"/></material>
+      </visual>
+      <collision>
+        <origin xyz="0.045 0 0" rpy="0 0 0"/>
+        <geometry><box size="0.09 0.018 0.03"/></geometry>
+      </collision>
+    </link>
+    <joint name="${name}_joint" type="revolute">
+      <origin xyz="0.025 ${reflect * 0.04} 0" rpy="0 0 0"/>
+      <parent link="gripper_base_link"/>
+      <child link="${name}_link"/>
+      <axis xyz="0 0 1"/>
+      <limit lower="-0.6" upper="0.6" effort="10" velocity="2.0"/>
+      <dynamics damping="0.05" friction="0.0"/>
+    </joint>
+  </xacro:macro>
+  <xacro:finger name="gripper_left"  reflect="1"/>
+  <xacro:finger name="gripper_right" reflect="-1"/>
+  <!-- Kontroler posisi per-jari (gz.msgs.Double, setpoint rad). -->
+  <gazebo>
+    <plugin filename="gz-sim-joint-position-controller-system"
+            name="gz::sim::systems::JointPositionController">
+      <joint_name>gripper_left_joint</joint_name>
+      <topic>hydroships/gripper_left/cmd</topic>
+      <p_gain>3.0</p_gain><i_gain>0.05</i_gain><d_gain>0.1</d_gain>
+    </plugin>
+  </gazebo>
+  <gazebo>
+    <plugin filename="gz-sim-joint-position-controller-system"
+            name="gz::sim::systems::JointPositionController">
+      <joint_name>gripper_right_joint</joint_name>
+      <topic>hydroships/gripper_right/cmd</topic>
+      <p_gain>3.0</p_gain><i_gain>0.05</i_gain><d_gain>0.1</d_gain>
+    </plugin>
+  </gazebo>
   <!-- ============================================================ -->
   <!-- ===================  Plugin Gazebo Fortress  =============== -->

Commit message: Add build logs and new mesh file for hydroships_gazebo
- Created command.log, stderr.log, stdout.log, stdout_stderr.log, streams.log, and logger_all.log to capture build process details for the hydroships_gazebo package.
- Added a new mesh file (rov.stl) to the hydroships_description package.

File: src/hydroships_description/urdf/hydroships.urdf.xacro (robot description, xacro)
@@ -35,8 +35,14 @@
                izz="${izz}"/>
     </inertial>
+    <!-- Visual: mesh ROV asli (meshes/rov.stl, hasil konversi model/rov.fbx →
+         di-decimate 1.26M → 40k tri, 2 MB; Fortress tak bisa FBX). Collision TETAP
+         kotak agar buoyancy graded & fisika tetap murah/stabil.
+         Skala 0.0048 menyamakan footprint mesh (~71 unit) ke ~0.345 m; origin
+         meng-offset agar mesh terpusat di base_link. Orientasi bow (yaw) & skala
+         mungkin perlu di-tune visual — lihat PROBLEM.md. -->
     <visual>
-      <origin xyz="0 0 0" rpy="0 0 0"/>
+      <origin xyz="-0.016 -0.068 0.002" rpy="0 0 0"/>
       <geometry>
-        <box size="${body_x} ${body_y} ${body_z}"/>
+        <mesh filename="package://hydroships_description/meshes/rov.stl" scale="0.0048 0.0048 0.0048"/>
       </geometry>
       <material name="hydro_yellow">
@@ -290,5 +296,8 @@
         <namespace>hydroships</namespace>
         <joint_name>${name}_joint</joint_name>
-        <topic>hydroships/${name}/thrust</topic>
+        <!-- namespace 'hydroships' di-prepend oleh plugin, jadi topic TANPA prefix
+             'hydroships/' -> subscribe ke /hydroships/${name}/thrust (cocok bridge).
+             Sebelumnya /hydroships/hydroships/... sehingga thrust TAK PERNAH masuk. -->
+        <topic>${name}/thrust</topic>
         <use_angvel_cmd>false</use_angvel_cmd>
         <fluid_density>${fluid_density}</fluid_density>

Commit message: Add build logs for hydroships_description package
- Created command.log to log build and install commands with their return statuses.
- Created stderr.log and stdout.log for capturing standard error and output during the build process.
- Created stdout_stderr.log to combine standard output and error logs.
- Created streams.log to log the timing and output of commands executed during the build.
- Created logger_all.log to capture detailed debug information and command execution flow for the build process.

File: src/hydroships_description/urdf/hydroships.urdf.xacro (robot description, xacro)
@@ -18,4 +18,7 @@
   <xacro:property name="body_y" value="0.345"/>
   <xacro:property name="body_z" value="0.286"/>
+  <!-- Rotasi yaw mesh visual (rad) agar haluan/bow menghadap +X (arah surge).
+       Sesuaikan bila bow mesh menghadap arah lain: 1.5708=+90°, -1.5708=-90°, 3.14159=180°. -->
+  <xacro:property name="bow_yaw" value="0"/>
   <!-- Massa base dipilih agar total near-neutral, sedikit positif buoyant. -->
   <xacro:property name="base_mass" value="33.6"/>
@@ -35,14 +38,13 @@
                izz="${izz}"/>
     </inertial>
-    <!-- Visual: mesh ROV asli (meshes/rov.stl, hasil konversi model/rov.fbx →
-         di-decimate 1.26M → 40k tri, 2 MB; Fortress tak bisa FBX). Collision TETAP
-         kotak agar buoyancy graded & fisika tetap murah/stabil.
-         Skala 0.0048 menyamakan footprint mesh (~71 unit) ke ~0.345 m; origin
-         meng-offset agar mesh terpusat di base_link. Orientasi bow (yaw) & skala
-         mungkin perlu di-tune visual — lihat PROBLEM.md. -->
+    <!-- Visual: mesh ROV asli (meshes/rov.stl, dari model/rov.fbx: node-transform
+         di-bake via PreTransformVertices lalu di-decimate; Fortress tak bisa FBX).
+         Mesh dalam MILIMETER (bbox 350.7 x 344.5 x 286 mm ≈ kotak desain) → scale 0.001.
+         Mesh sudah di-center di file, jadi origin xyz=0. rpy=0 0 ${bow_yaw}: arah bow
+         (+X) mungkin perlu diputar — lihat PROBLEM.md. Collision TETAP kotak (fisika). -->
     <visual>
-      <origin xyz="-0.016 -0.068 0.002" rpy="0 0 0"/>
+      <origin xyz="0 0 0" rpy="0 0 ${bow_yaw}"/>
       <geometry>
-        <mesh filename="package://hydroships_description/meshes/rov.stl" scale="0.0048 0.0048 0.0048"/>
+        <mesh filename="package://hydroships_description/meshes/rov.stl" scale="0.001 0.001 0.001"/>
       </geometry>
       <material name="hydro_yellow">

Commit message: Enhance thruster macro in hydroships.urdf.xacro with visual properties and adjust thruster dimensions for improved accuracy

File: src/hydroships_description/urdf/hydroships.urdf.xacro (robot description, xacro)
@@ -66,5 +66,5 @@
     axis  : arah dorong (unit vector) di frame body; juga sumbu putar propeller
   -->
-  <xacro:macro name="thruster" params="name xyz axis">
+  <xacro:macro name="thruster" params="name xyz axis visual_rpy='0 0 0' visual_offset='0 0 0'">
     <link name="${name}">
       <inertial>
@@ -75,10 +75,19 @@
       </inertial>
       <visual>
-        <origin xyz="0 0 0" rpy="0 0 0"/>
+        <origin xyz="${visual_offset}" rpy="${visual_rpy}"/>
         <geometry>
-          <cylinder radius="0.02" length="0.06"/>
+          <cylinder radius="0.012" length="0.05"/>
         </geometry>
         <material name="hydro_dark">
           <color rgba="0.1 0.1 0.12 1.0"/>
+        </material>
+      </visual>
+      <visual>
+        <origin xyz="${visual_offset}" rpy="${visual_rpy}"/>
+        <geometry>
+          <cylinder radius="0.024" length="0.008"/>
+        </geometry>
+        <material name="hydro_yellow">
+          <color rgba="0.9 0.75 0.1 1.0"/>
         </material>
       </visual>
@@ -103,10 +112,10 @@
          thruster_5 = T100-B (lateral bawah horizontal)
          thruster_6 = T100-D (belakang sentral vertikal) -->
-    <xacro:thruster name="thruster_1" xyz="0.1234 0.0275 0.0142" axis="0.0 0.0 1.0"/>
-    <xacro:thruster name="thruster_2" xyz="-0.1228 0.0290 0.0148" axis="0.0 0.0 1.0"/>
-    <xacro:thruster name="thruster_3" xyz="0.1371 -0.1298 0.0336" axis="1.0 0.0 0.0"/>
-    <xacro:thruster name="thruster_4" xyz="-0.1371 -0.1296 0.0374" axis="1.0 0.0 0.0"/>
-    <xacro:thruster name="thruster_5" xyz="0.0003 0.0455 -0.0994" axis="0.0 1.0 0.0"/>
-    <xacro:thruster name="thruster_6" xyz="-0.0003 0.1364 0.0403" axis="0.0 0.0 1.0"/>
+    <xacro:thruster name="thruster_1" xyz="0.1234 0.0275 0.0142" axis="0.0 0.0 1.0" visual_rpy="0 1.5708 0" visual_offset="0.008 0.004 0.000"/>
+    <xacro:thruster name="thruster_2" xyz="-0.1228 0.0290 0.0148" axis="0.0 0.0 1.0" visual_rpy="0 1.5708 0" visual_offset="0.008 -0.004 0.000"/>
+    <xacro:thruster name="thruster_3" xyz="0.1371 -0.1298 0.0336" axis="1.0 0.0 0.0" visual_rpy="1.5708 0 0" visual_offset="0.008 -0.002 -0.002"/>
+    <xacro:thruster name="thruster_4" xyz="-0.1371 -0.1296 0.0374" axis="1.0 0.0 0.0" visual_rpy="1.5708 0 0" visual_offset="0.008 0.002 -0.002"/>
+    <xacro:thruster name="thruster_5" xyz="0.0003 0.0455 -0.0994" axis="0.0 1.0 0.0" visual_rpy="0 0 1.5708" visual_offset="0.000 0.000 0.008"/>
+    <xacro:thruster name="thruster_6" xyz="-0.0003 0.1364 0.0403" axis="0.0 0.0 1.0" visual_rpy="0 1.5708 0" visual_offset="0.006 0.000 -0.001"/>
   <!-- ==================== Frame sensor (placeholder M3) ==================== -->
   <link name="imu_link"/>

Commit message: feat(urdf): enhance body gripper visibility and physical properties
Increase the scale, mass, and visual contrast of the body gripper
components in the URDF to ensure they are clearly visible and
physically representative in Gazebo simulations.

- Resize `gripper_base` from 0.05m³ to 0.08x0.08x0.10m
- Update `gripper_base` mass to 0.12kg and adjust inertia
- Change `gripper_base` material to a high-contrast yellow
- Adjust `gripper_base_joint` offset to `xyz="0.08 0 -0.22"`
- Resize `gripper_jaw` to 0.016x0.04x0.10m for better visual feedback
- Update documentation (CHANGELOG, HOW-TO-RUN, STATUS) to reflect
  new gripper dimensions and verification steps

File: src/hydroships_description/urdf/hydroships.urdf.xacro (robot description, xacro)
@@ -248,24 +248,26 @@
        (indikator visual buka/tutup). Reach ke BAWAH dari perut ROV karena
        payload di-approach dari atas (kamera bawah). Lihat PROBLEM.md. -->
-  <xacro:property name="grip_mass" value="0.05"/>
-  <!-- Pangkal gripper: menempel kaku di perut depan ROV, menghadap ke bawah. -->
+  <!-- Pangkal gripper: menempel kaku di perut depan ROV, menghadap ke bawah.
+       Body gripper diperbesar agar terlihat di Gazebo dan memiliki massa yang masuk akal
+       untuk interaksi DetachableJoint dengan payload. -->
+  <xacro:property name="grip_mass" value="0.12"/>
   <link name="gripper_base">
     <inertial>
       <origin xyz="0 0 0" rpy="0 0 0"/>
       <mass value="${grip_mass}"/>
-      <inertia ixx="1e-4" ixy="0.0" ixz="0.0" iyy="1e-4" iyz="0.0" izz="1e-4"/>
+      <inertia ixx="2.6e-4" ixy="0.0" ixz="0.0" iyy="2.6e-4" iyz="0.0" izz="3.3e-4"/>
     </inertial>
     <visual>
       <origin xyz="0 0 0" rpy="0 0 0"/>
-      <geometry><box size="0.05 0.05 0.03"/></geometry>
-      <material name="hydro_grip"><color rgba="0.2 0.2 0.22 1.0"/></material>
+      <geometry><box size="0.08 0.08 0.10"/></geometry>
+      <material name="hydro_grip"><color rgba="0.85 0.7 0.1 1.0"/></material>
     </visual>
     <collision>
       <origin xyz="0 0 0" rpy="0 0 0"/>
-      <geometry><box size="0.05 0.05 0.03"/></geometry>
+      <geometry><box size="0.08 0.08 0.10"/></geometry>
     </collision>
   </link>
   <joint name="gripper_base_joint" type="fixed">
-    <origin xyz="0.06 0 -0.16" rpy="0 0 0"/>
+    <origin xyz="0.08 0 -0.22" rpy="0 0 0"/>
     <parent link="base_link"/>
     <child link="gripper_base"/>
@@ -280,19 +282,24 @@
     <preserveFixedJoint>true</preserveFixedJoint>
   </gazebo>
-  <!-- Jari tunggal (1 DOF revolute, sumbu y). Kosmetik: menandai buka/tutup. -->
+  <!-- Jari tunggal (1 DOF revolute, sumbu y). Kosmetik: menandai buka/tutup.
+       Diperbesar agar posisi buka/tutup terlihat jelas di Gazebo. -->
   <link name="gripper_jaw">
     <inertial>
-      <origin xyz="0 0 -0.03" rpy="0 0 0"/>
+      <origin xyz="0 0 -0.05" rpy="0 0 0"/>
       <mass value="${grip_mass}"/>
-      <inertia ixx="1e-4" ixy="0.0" ixz="0.0" iyy="1e-4" iyz="0.0" izz="1e-4"/>
+      <inertia ixx="2.0e-5" ixy="0.0" ixz="0.0" iyy="2.0e-5" iyz="0.0" izz="2.5e-5"/>
     </inertial>
     <visual>
-      <origin xyz="0 0 -0.03" rpy="0 0 0"/>
-      <geometry><box size="0.012 0.03 0.06"/></geometry>
-      <material name="hydro_jaw"><color rgba="0.85 0.7 0.1 1.0"/></material>
-    </visual>
+      <origin xyz="0 0 -0.05" rpy="0 0 0"/>
+      <geometry><box size="0.016 0.04 0.10"/></geometry>
+      <material name="hydro_jaw"><color rgba="0.95 0.8 0.2 1.0"/></material>
+    </visual>
+    <collision>
+      <origin xyz="0 0 -0.05" rpy="0 0 0"/>
+      <geometry><box size="0.016 0.04 0.10"/></geometry>
+    </collision>
   </link>
   <joint name="gripper_jaw_joint" type="revolute">
-    <origin xyz="0.02 0 -0.015" rpy="0 0 0"/>
+    <origin xyz="0.04 0 -0.04" rpy="0 0 0"/>
     <parent link="gripper_base"/>
     <child link="gripper_jaw"/>

Commit message: refactor(urdf): relocate body gripper to front mount
Relocate the body gripper from the bottom belly of the ROV to the
front face (+X direction) to align with the physical design
specifications.

- Update `gripper_base_joint` origin to `0.18 0 0` for front mounting
- Redesign `gripper_base` geometry to `0.10 0.10 0.06` m
- Reorient `gripper_jaw` to extend forward (+X) with new dimensions
  of `0.12 0.016 0.04` m
- Adjust inertial properties and collision boxes for the new
  geometry and mounting position
- Update documentation (CHANGELOG, HOW-TO-RUN, STATUS) and internal
  planning files to reflect the new mounting configuration

File: src/hydroships_description/urdf/hydroships.urdf.xacro (robot description, xacro)
@@ -246,28 +246,26 @@
        lolos uji grasp). Grasp FISIK memakai gz-sim DetachableJoint (sambungan
        kaku ROV<->payload), BUKAN gesekan jari. Jari tunggal di sini KOSMETIK
-       (indikator visual buka/tutup). Reach ke BAWAH dari perut ROV karena
-       payload di-approach dari atas (kamera bawah). Lihat PROBLEM.md. -->
-  <!-- Pangkal gripper: menempel kaku di perut depan ROV, menghadap ke bawah.
-       Body gripper diperbesar agar terlihat di Gazebo dan memiliki massa yang masuk akal
-       untuk interaksi DetachableJoint dengan payload. -->
+       (indikator visual buka/tutup). Dipasang di MUKA DEPAN ROV, menjorok
+       ke arah depan (+X). Lihat PROBLEM.md. -->
   <xacro:property name="grip_mass" value="0.12"/>
+  <!-- Body gripper di muka depan ROV, menjorok ke depan (+X). -->
   <link name="gripper_base">
     <inertial>
       <origin xyz="0 0 0" rpy="0 0 0"/>
       <mass value="${grip_mass}"/>
-      <inertia ixx="2.6e-4" ixy="0.0" ixz="0.0" iyy="2.6e-4" iyz="0.0" izz="3.3e-4"/>
+      <inertia ixx="1.4e-4" ixy="0.0" ixz="0.0" iyy="1.4e-4" iyz="0.0" izz="2.0e-4"/>
     </inertial>
     <visual>
       <origin xyz="0 0 0" rpy="0 0 0"/>
-      <geometry><box size="0.08 0.08 0.10"/></geometry>
+      <geometry><box size="0.10 0.10 0.06"/></geometry>
       <material name="hydro_grip"><color rgba="0.85 0.7 0.1 1.0"/></material>
     </visual>
     <collision>
       <origin xyz="0 0 0" rpy="0 0 0"/>
-      <geometry><box size="0.08 0.08 0.10"/></geometry>
+      <geometry><box size="0.10 0.10 0.06"/></geometry>
     </collision>
   </link>
   <joint name="gripper_base_joint" type="fixed">
-    <origin xyz="0.08 0 -0.22" rpy="0 0 0"/>
+    <origin xyz="0.18 0 0" rpy="0 0 0"/>
     <parent link="base_link"/>
     <child link="gripper_base"/>
@@ -283,23 +281,23 @@
   </gazebo>
   <!-- Jari tunggal (1 DOF revolute, sumbu y). Kosmetik: menandai buka/tutup.
-       Diperbesar agar posisi buka/tutup terlihat jelas di Gazebo. -->
+       Jari menjorok ke depan (+X) dari body gripper. -->
   <link name="gripper_jaw">
     <inertial>
-      <origin xyz="0 0 -0.05" rpy="0 0 0"/>
+      <origin xyz="0.06 0 0" rpy="0 0 0"/>
       <mass value="${grip_mass}"/>
-      <inertia ixx="2.0e-5" ixy="0.0" ixz="0.0" iyy="2.0e-5" iyz="0.0" izz="2.5e-5"/>
+      <inertia ixx="1.9e-4" ixy="0.0" ixz="0.0" iyy="8.5e-7" iyz="0.0" izz="1.9e-4"/>
     </inertial>
     <visual>
-      <origin xyz="0 0 -0.05" rpy="0 0 0"/>
-      <geometry><box size="0.016 0.04 0.10"/></geometry>
+      <origin xyz="0 0 0" rpy="0 0 0"/>
+      <geometry><box size="0.12 0.016 0.04"/></geometry>
       <material name="hydro_jaw"><color rgba="0.95 0.8 0.2 1.0"/></material>
     </visual>
     <collision>
-      <origin xyz="0 0 -0.05" rpy="0 0 0"/>
-      <geometry><box size="0.016 0.04 0.10"/></geometry>
+      <origin xyz="0 0 0" rpy="0 0 0"/>
+      <geometry><box size="0.12 0.016 0.04"/></geometry>
     </collision>
   </link>
   <joint name="gripper_jaw_joint" type="revolute">
-    <origin xyz="0.04 0 -0.04" rpy="0 0 0"/>
+    <origin xyz="0.05 0 0" rpy="0 0 0"/>
     <parent link="gripper_base"/>
     <child link="gripper_jaw"/>
