Commit message: New Model Gripper

File: src/hydroships_description/urdf/hydroships.urdf.xacro (robot description, xacro)
@@ -243,9 +243,8 @@
   </gazebo>
   <!-- ==================== Manipulator (rancang ulang M5) ====================
-       Gripper 1-DOF SEDERHANA (bukan 2 jari kompleks versi lama yg tak pernah
-       lolos uji grasp). Grasp FISIK memakai gz-sim DetachableJoint (sambungan
-       kaku ROV<->payload), BUKAN gesekan jari. Jari tunggal di sini KOSMETIK
-       (indikator visual buka/tutup). Dipasang di MUKA DEPAN ROV, menjorok
-       ke arah depan (+X). Lihat PROBLEM.md. -->
+       Grasp FISIK memakai gz-sim DetachableJoint (sambungan kaku ROV<->payload),
+       BUKAN gesekan jari. DUA JARI opposing (kiri/kanan) di sini KOSMETIK
+       (indikator visual buka/tutup) — digerakkan SEREMPAK dari satu nilai sudut.
+       Dipasang di MUKA DEPAN ROV, menjorok ke arah depan (+X). Lihat PROBLEM.md. -->
   <xacro:property name="grip_mass" value="0.12"/>
   <!-- Body gripper di muka depan ROV, menjorok ke depan (+X). -->
@@ -280,30 +279,38 @@
     <preserveFixedJoint>true</preserveFixedJoint>
   </gazebo>
-  <!-- Jari tunggal (1 DOF revolute, sumbu y). Kosmetik: menandai buka/tutup.
-       Jari menjorok ke depan (+X) dari body gripper. -->
-  <link name="gripper_jaw">
-    <inertial>
-      <origin xyz="0.06 0 0" rpy="0 0 0"/>
-      <mass value="${grip_mass}"/>
-      <inertia ixx="1.9e-4" ixy="0.0" ixz="0.0" iyy="8.5e-7" iyz="0.0" izz="1.9e-4"/>
-    </inertial>
-    <visual>
-      <origin xyz="0 0 0" rpy="0 0 0"/>
-      <geometry><box size="0.12 0.016 0.04"/></geometry>
-      <material name="hydro_jaw"><color rgba="0.95 0.8 0.2 1.0"/></material>
-    </visual>
-    <collision>
-      <origin xyz="0 0 0" rpy="0 0 0"/>
-      <geometry><box size="0.12 0.016 0.04"/></geometry>
-    </collision>
-  </link>
-  <joint name="gripper_jaw_joint" type="revolute">
-    <origin xyz="0.05 0 0" rpy="0 0 0"/>
-    <parent link="gripper_base"/>
-    <child link="gripper_jaw"/>
-    <axis xyz="0 1 0"/>
-    <limit lower="-0.1" upper="1.2" effort="10.0" velocity="2.0"/>
-    <dynamics damping="0.05" friction="0.0"/>
-  </joint>
+  <!-- Dua jari opposing (masing-masing 1 DOF revolute, sumbu Z) -> menjepit di
+       bidang XY seperti parallel gripper pada umumnya. Kosmetik: menandai
+       buka/tutup. Sudut 0 = TERTUTUP (kedua jari sejajar menghadap +X); sudut
+       naik = MEMBUKA (tip menjauh dari sumbu tengah). Mirroring diurus tanda
+       axis (kiri 0 0 -1, kanan 0 0 1) sehingga nilai Float64 yang SAMA dikirim
+       ke kedua joint dan gerakannya otomatis simetris. -->
+  <xacro:macro name="gripper_finger" params="side y_pivot axis_z">
+    <link name="gripper_finger_${side}">
+      <inertial>
+        <origin xyz="0.04 0 0" rpy="0 0 0"/>
+        <mass value="0.06"/>
+        <inertia ixx="6.0e-6" ixy="0.0" ixz="0.0" iyy="3.6e-5" iyz="0.0" izz="3.4e-5"/>
+      </inertial>
+      <visual>
+        <origin xyz="0.04 0 0" rpy="0 0 0"/>
+        <geometry><box size="0.08 0.016 0.03"/></geometry>
+        <material name="hydro_jaw"><color rgba="0.95 0.8 0.2 1.0"/></material>
+      </visual>
+      <collision>
+        <origin xyz="0.04 0 0" rpy="0 0 0"/>
+        <geometry><box size="0.08 0.016 0.03"/></geometry>
+      </collision>
+    </link>
+    <joint name="gripper_${side}_joint" type="revolute">
+      <origin xyz="0.04 ${y_pivot} 0" rpy="0 0 0"/>
+      <parent link="gripper_base"/>
+      <child link="gripper_finger_${side}"/>
+      <axis xyz="0 0 ${axis_z}"/>
+      <limit lower="-0.1" upper="0.5" effort="10.0" velocity="2.0"/>
+      <dynamics damping="0.05" friction="0.0"/>
+    </joint>
+  </xacro:macro>
+  <xacro:gripper_finger side="left"  y_pivot="-0.025" axis_z="-1"/>
+  <xacro:gripper_finger side="right" y_pivot="0.025"  axis_z="1"/>
   <!-- ============================================================ -->
   <!-- ===================  Plugin Gazebo Fortress  =============== -->
@@ -383,16 +390,22 @@
   <xacro:thruster_plugin name="thruster_6" diameter="0.048"/>
   <!-- ============ Plugin manipulator (rancang ulang M5) ============ -->
-  <!-- Kontrol posisi jari kosmetik: target sudut (rad) via gz.msgs.Double di
-       /hydroships/gripper_jaw/cmd (dijembatani dari ROS Float64). -->
-  <gazebo>
-    <plugin filename="gz-sim-joint-position-controller-system"
-            name="gz::sim::systems::JointPositionController">
-      <joint_name>gripper_jaw_joint</joint_name>
-      <topic>/hydroships/gripper_jaw/cmd</topic>
-      <p_gain>2.0</p_gain>
-      <i_gain>0.0</i_gain>
-      <d_gain>0.1</d_gain>
-    </plugin>
-  </gazebo>
+  <!-- Kontrol posisi dua jari kosmetik: target sudut (rad) via gz.msgs.Double di
+       /hydroships/gripper_left/cmd & /hydroships/gripper_right/cmd (dijembatani
+       dari ROS Float64). Satu instance plugin per joint (cara standar Fortress);
+       nilai yang dikirim identik, mirroring dari tanda axis di URDF. -->
+  <xacro:macro name="gripper_finger_plugin" params="side">
+    <gazebo>
+      <plugin filename="gz-sim-joint-position-controller-system"
+              name="gz::sim::systems::JointPositionController">
+        <joint_name>gripper_${side}_joint</joint_name>
+        <topic>/hydroships/gripper_${side}/cmd</topic>
+        <p_gain>2.0</p_gain>
+        <i_gain>0.0</i_gain>
+        <d_gain>0.1</d_gain>
+      </plugin>
+    </gazebo>
+  </xacro:macro>
+  <xacro:gripper_finger_plugin side="left"/>
+  <xacro:gripper_finger_plugin side="right"/>
   <!-- GRASP FISIK: DetachableJoint membuat sambungan kaku gripper_base<->payload.
        attach saat pesan di /hydroships/gripper/attach, detach di .../detach

Commit message: Konversi F3Z ke URDF

File: src/hydroships_description/urdf/hydroships.urdf.xacro (robot description, xacro)
@@ -4,10 +4,23 @@
   Frame konvensi ROS (REP-103): x maju (surge), y kiri (sway), z atas (heave).
   Catatan penyederhanaan M1:
-    * Rangka dimodelkan sebagai satu kotak solid 0.345 x 0.345 x 0.286 m.
-      Volume perpindahan air kotak ~0.0340 m^3 -> gaya apung setara ~34.05 kg.
-      Massa total (base + 6 thruster) dibuat SEDIKIT DI BAWAH itu supaya ROV
-      apung pelan saat thruster mati (near-neutral, sedikit positif).
-      Ini placeholder yang di-tune di M2, BUKAN massa ROV asli.
+    * Visual tetap primitif (box/cylinder) supaya ringan; lihat
+      rov_kki2026_new_design.urdf.xacro untuk versi bermesh CAD.
     * Koefisien hidrodinamika memakai nilai acuan tipe BlueROV2 (di-tune belakangan).
+  DISINKRONKAN DENGAN CAD (2026-07-28)
+    Dimensi, posisi/sumbu thruster, massa, inertia, dan volume collision kini
+    diturunkan dari "DOKUMENTASI ROV/@ROV KKI 2026 NEW DESIGN.stl" lewat
+    hydroships_description/scripts/measure_cad_frames.py, dan penomoran
+    thruster mengikuti Gambar 2.9/2.10 dokumen desain (penulis, 2026).
+    Model ini dan rov_kki2026_new_design.urdf.xacro kini memakai geometri
+    thruster, massa, dan inertia yang IDENTIK — bedanya hanya visual
+    (primitif vs mesh CAD). allocation.py sudah ikut disinkronkan.
+    Volume collision SENGAJA jauh lebih kecil dari bbox: ROV ini rangka
+    TERBUKA, air mengalir menembusnya, jadi volume air yang benar-benar
+    tergeser hanya 0.006644 m^3 (bahan padat + rongga tabung enclosure),
+    bukan 0.0508 m^3 seperti kotak penuh. Kotak collision di bawah disetel
+    agar volumenya tepat sama dgn angka terukur itu, dan pusatnya 0.02 m di
+    atas CoG supaya CoB > CoG (stabil). Konsekuensi: saat menyentuh dasar
+    kolam, badan ROV akan tampak tenggelam sebagian ke lantai — itu harga
+    dari apung yang benar. Lihat rov_kki2026_new_design.parts.md.
   PARAMETER FISIK TER-EKSTERNAL: massa, CoG/CoB, tensor inertia, & 18 koefisien
   hidrodinamika kini dibaca dari config/rov_params.yaml (via xacro.load_yaml)
@@ -20,7 +33,11 @@
 <robot name="hydroships" xmlns:xacro="http://www.ros.org/wiki/xacro">
   <!-- ============================ Parameter ============================ -->
-  <xacro:property name="body_x" value="0.345"/>
-  <xacro:property name="body_y" value="0.345"/>
-  <xacro:property name="body_z" value="0.286"/>
+  <!-- bbox ROV terukur dari CAD (m). -->
+  <xacro:property name="body_x" value="0.5079"/>
+  <xacro:property name="body_y" value="0.3469"/>
+  <xacro:property name="body_z" value="0.2959"/>
+  <!-- Kotak collision = volume air TERGESER terukur (0.006644 m^3), bukan bbox.
+       Tebal = 0.006644 / (body_x * body_y). Pusat 0.02 m di atas CoG. -->
+  <xacro:property name="cob_z" value="0.02"/>
   <!-- (bow_yaw dulu untuk memutar mesh; visual kini primitif dgn haluan tetap +X.) -->
   <!-- ===== Parameter FISIK dari config/rov_params.yaml =====================
@@ -32,6 +49,17 @@
        (share/pkg/urdf), keduanya bersebelahan dgn .../config. -->
   <xacro:property name="rp" value="${xacro.load_yaml('../config/rov_params.yaml')}"/>
-  <xacro:property name="base_mass" value="${rp['base_mass']}"/>
+  <xacro:property name="vehicle_mass" value="${rp['vehicle_mass']}"/>
+  <xacro:property name="displaced_volume" value="${rp['displaced_volume']}"/>
   <xacro:property name="thruster_mass" value="${rp['thruster_mass']}"/>
+  <!-- Massa link tambahan model ini (gripper + 2 jari + 6 thruster). base_link
+       mendapat sisanya, supaya massa TOTAL = vehicle_mass persis sama dengan
+       rov_kki2026_new_design.urdf.xacro meski link tambahannya berbeda. -->
+  <xacro:property name="grip_mass" value="0.12"/>
+  <xacro:property name="finger_mass" value="0.06"/>
+  <xacro:property name="aux_mass" value="${6*thruster_mass + grip_mass + 2*finger_mass}"/>
+  <xacro:property name="base_mass" value="${vehicle_mass - aux_mass}"/>
+  <!-- Volume collision link tambahan; dikurangkan dari kotak base_link supaya
+       TOTAL volume collision = displaced_volume terukur. -->
+  <xacro:property name="aux_volume" value="${0.10*0.10*0.06 + 2*(0.08*0.016*0.03)}"/>
   <xacro:property name="fluid_density" value="${rp['fluid_density']}"/>
   <xacro:property name="cog" value="${rp['cog']}"/>
@@ -102,9 +130,10 @@
       </material>
     </visual>
-    <!-- Collision box dipakai plugin Buoyancy untuk menghitung volume perpindahan. -->
+    <!-- Collision box dipakai plugin Buoyancy untuk menghitung volume perpindahan.
+         Ukurannya = volume tergeser terukur, BUKAN bbox (lihat header). -->
     <collision>
-      <origin xyz="0 0 0" rpy="0 0 0"/>
+      <origin xyz="0 0 ${cob_z}" rpy="0 0 0"/>
       <geometry>
-        <box size="${body_x} ${body_y} ${body_z}"/>
+        <box size="${body_x} ${body_y} ${(displaced_volume - aux_volume) / (body_x * body_y)}"/>
       </geometry>
     </collision>
@@ -154,25 +183,30 @@
     </joint>
   </xacro:macro>
-    <!-- ==================== Thruster positions (dari thruster_positions.csv) ==========
-         Posisi di FRAME BODY ROS (x=maju, y=kiri, z=atas), dikonversi dari CSV
-         (X=lateral kanan+, Y=fore/aft DEPAN negatif, Z=atas) via:
-             x_body = -Y_csv,  y_body = -X_csv,  z_body = Z_csv.
-         HARUS konsisten dgn hydroships_control/allocation.py (THRUSTERS).
-         (Perbaikan: dulu kolom CSV disalin mentah -> posisi terputar 90° -> yaw
-          near-singular. Setelah dikoreksi cond TAM ~20, yaw pulih. Lihat PROBLEM.md.)
-         Mapping & peran:
-           thruster_1 = T200-E (vertikal, kanan)
-           thruster_2 = T200-F (vertikal, kiri)
-           thruster_3 = T100-C (surge, depan-kanan)
-           thruster_4 = T100-A (surge, depan-kiri)
-           thruster_5 = T200-B (sway/menyamping, tengah-bawah)   [eks label T100-B]
-           thruster_6 = T100-D (vertikal, belakang-tengah)
-         Catatan: visual_rpy/visual_offset hanya kosmetik (orientasi silinder hias). -->
-    <xacro:thruster name="thruster_1" xyz="-0.0275 -0.1234 0.0142" axis="0.0 0.0 1.0" visual_rpy="0 0 0" visual_offset="0 0 0.008"/>
-    <xacro:thruster name="thruster_2" xyz="-0.0290 0.1228 0.0148" axis="0.0 0.0 1.0" visual_rpy="0 0 0" visual_offset="0 0 0.008"/>
-    <xacro:thruster name="thruster_3" xyz="0.1298 -0.1371 0.0336" axis="1.0 0.0 0.0" visual_rpy="0 1.5708 0" visual_offset="0.008 0 0"/>
-    <xacro:thruster name="thruster_4" xyz="0.1296 0.1371 0.0374" axis="1.0 0.0 0.0" visual_rpy="0 1.5708 0" visual_offset="0.008 0 0"/>
-    <xacro:thruster name="thruster_5" xyz="-0.0455 -0.0003 -0.0994" axis="0.0 1.0 0.0" visual_rpy="1.5708 0 0" visual_offset="0 0.008 0"/>
-    <xacro:thruster name="thruster_6" xyz="-0.1364 0.0003 0.0403" axis="0.0 0.0 1.0" visual_rpy="0 0 0" visual_offset="0 0 0.008"/>
+    <!-- ==================== Thruster positions (TERUKUR dari CAD) ==========
+         Posisi & sumbu diukur dari @ROV KKI 2026 NEW DESIGN.stl via
+         scripts/measure_cad_frames.py; penomoran mengikuti Gambar 2.9/2.10
+         dokumen desain (penulis, 2026). HARUS konsisten dgn
+         hydroships_control/allocation.py (THRUSTERS) dan docs/thruster_config.md.
+           nama        peran               kelas  duct terukur
+           thruster_1  surge kanan         T200   duct 90.1 mm
+           thruster_2  surge kiri          T200   duct 90.1 mm
+           thruster_3  heave haluan kanan  T100   prop 66.6 mm
+           thruster_4  heave haluan kiri   T100   prop 66.6 mm
+           thruster_5  heave buritan       T100   prop 66.6 mm
+           thruster_6  sway tengah-bawah   T100   prop 59.0 mm
+         Mapping LAMA menukar peran pasangan haluan <-> tengah (1,2 dikira
+         vertikal, 3,4 surge) dan menukar 5 <-> 6. CAD & Gambar 2.9 keduanya
+         menunjukkan sebaliknya. Setelah koreksi, cond(TAM) 19.7 -> 10.0 dan
+         gaya thruster utk wrench satuan pada DOF terlemah 9.25 N -> 4.06 N.
+         Arah putar propeller (Gambar 2.9): 1=CCW 2=CW 3=CCW 4=CW 5=CW 6=CCW
+         — tiap pasangan berlawanan agar torsi reaksi saling meniadakan.
+         Tanda sumbu masih perlu verifikasi bench (lihat allocation.py).
+         Catatan: visual_rpy/visual_offset hanya kosmetik. -->
+    <xacro:thruster name="thruster_1" xyz="-0.0291 -0.1188 0.0186" axis="1.0 0.0 0.0" visual_rpy="0 1.5708 0" visual_offset="0.008 0 0"/>
+    <xacro:thruster name="thruster_2" xyz="-0.0287 0.1274 0.0190"  axis="1.0 0.0 0.0" visual_rpy="0 1.5708 0" visual_offset="0.008 0 0"/>
+    <xacro:thruster name="thruster_3" xyz="0.1050 -0.1332 0.0592"  axis="0.0 0.0 1.0" visual_rpy="0 0 0"      visual_offset="0 0 0.008"/>
+    <xacro:thruster name="thruster_4" xyz="0.1053 0.1411 0.0550"   axis="0.0 0.0 1.0" visual_rpy="0 0 0"      visual_offset="0 0 0.008"/>
+    <xacro:thruster name="thruster_5" xyz="-0.1610 0.0037 0.0621"  axis="0.0 0.0 1.0" visual_rpy="0 0 0"      visual_offset="0 0 0.008"/>
+    <xacro:thruster name="thruster_6" xyz="-0.0700 0.0200 -0.0939" axis="0.0 1.0 0.0" visual_rpy="1.5708 0 0" visual_offset="0 0.008 0"/>
   <!-- ==================== Frame sensor (placeholder M3) ==================== -->
   <link name="imu_link"/>
@@ -247,5 +281,4 @@
        (indikator visual buka/tutup) — digerakkan SEREMPAK dari satu nilai sudut.
        Dipasang di MUKA DEPAN ROV, menjorok ke arah depan (+X). Lihat PROBLEM.md. -->
-  <xacro:property name="grip_mass" value="0.12"/>
   <!-- Body gripper di muka depan ROV, menjorok ke depan (+X). -->
   <link name="gripper_base">
@@ -289,5 +322,5 @@
       <inertial>
         <origin xyz="0.04 0 0" rpy="0 0 0"/>
-        <mass value="0.06"/>
+        <mass value="${finger_mass}"/>
         <inertia ixx="6.0e-6" ixy="0.0" ixz="0.0" iyy="3.6e-5" iyz="0.0" izz="3.4e-5"/>
       </inertial>
@@ -382,11 +415,14 @@
     </gazebo>
   </xacro:macro>
-  <!-- Horizontal ~ diameter 0.076 (kelas T200); vertikal ~ 0.048 (kelas T100). -->
-  <xacro:thruster_plugin name="thruster_1" diameter="0.076"/>
-  <xacro:thruster_plugin name="thruster_2" diameter="0.076"/>
-  <xacro:thruster_plugin name="thruster_3" diameter="0.076"/>
-  <xacro:thruster_plugin name="thruster_4" diameter="0.048"/>
-  <xacro:thruster_plugin name="thruster_5" diameter="0.048"/>
-  <xacro:thruster_plugin name="thruster_6" diameter="0.048"/>
+  <!-- Diameter mengikuti KELAS hasil ukur CAD: T200 (surge) duct 90 mm ->
+       0.076 m; T100 (heave & sway) prop 66.6 mm -> 0.048 m. Sebelumnya
+       pembagian 0.076/0.048 mengikuti nomor urut, bukan kelas, sehingga
+       dua unit identik bisa dapat diameter berbeda. -->
+  <xacro:thruster_plugin name="thruster_1" diameter="0.076"/>  <!-- T200 surge -->
+  <xacro:thruster_plugin name="thruster_2" diameter="0.076"/>  <!-- T200 surge -->
+  <xacro:thruster_plugin name="thruster_3" diameter="0.048"/>  <!-- T100 heave -->
+  <xacro:thruster_plugin name="thruster_4" diameter="0.048"/>  <!-- T100 heave -->
+  <xacro:thruster_plugin name="thruster_5" diameter="0.048"/>  <!-- T100 heave -->
+  <xacro:thruster_plugin name="thruster_6" diameter="0.048"/>  <!-- T100 sway  -->
   <!-- ============ Plugin manipulator (rancang ulang M5) ============ -->
   <!-- Kontrol posisi dua jari kosmetik: target sudut (rad) via gz.msgs.Double di

Commit message: chore(physics): update mass properties and buoyancy compensation
Adjust the ROV base mass from 33.6kg to 8.3kg to reflect measured values,
consequently updating the inertia tensor and gripper mass properties.

Due to the significantly reduced mass while maintaining the same hull
volume, the net buoyancy has increased to ~+248.6N. The vertical
buoyancy feedforward is capped at -120.0N to match the maximum physical
thrust capacity of the vertical thrusters, acknowledging that the ROV
will remain positively buoyant until physical ballast is added.

File: src/hydroships_description/urdf/hydroships.urdf.xacro (robot description, xacro)
@@ -250,5 +250,5 @@
        (indikator visual buka/tutup) — digerakkan SEREMPAK dari satu nilai sudut.
        Dipasang di MUKA DEPAN ROV, menjorok ke arah depan (+X). Lihat PROBLEM.md. -->
-  <xacro:property name="grip_mass" value="0.12"/>
+  <xacro:property name="grip_mass" value="0.08"/>
   <!-- Body gripper di muka depan ROV, menjorok ke depan (+X). -->
   <link name="gripper_base">
@@ -292,5 +292,5 @@
       <inertial>
         <origin xyz="0.04 0 0" rpy="0 0 0"/>
-        <mass value="0.06"/>
+        <mass value="0.01"/>
         <inertia ixx="6.0e-6" ixy="0.0" ixz="0.0" iyy="3.6e-5" iyz="0.0" izz="3.4e-5"/>
       </inertial>

Commit message: feat(physics): scale buoyancy volume and hydrodynamic coefficients
Implement a scaled collision box for buoyancy calculations to achieve
near-neutral buoyancy (~+0.28N) with the updated 8.3kg base mass. This
replaces the previous full-body bounding box approach which caused
excessive upward force.

Additionally, scale all hydrodynamic coefficients (added mass, linear
damping, and quadratic damping) by a factor of ~0.247 to maintain
proportionality with the reduced vehicle mass and prevent numerical
instability in the physics solver.

- Update `buoyancy_ff` from -120.0 to -0.3 in controller gains
- Define `buoyancy_collision` dimensions in `rov_params.yaml`
- Apply scaled coefficients to Fossen model parameters
- Update URDF to use scaled collision geometry for buoyancy volume

File: src/hydroships_description/urdf/hydroships.urdf.xacro (robot description, xacro)
@@ -4,8 +4,11 @@
   Frame konvensi ROS (REP-103): x maju (surge), y kiri (sway), z atas (heave).
   Catatan penyederhanaan M1:
-    * Rangka dimodelkan sebagai satu kotak solid 0.345 x 0.345 x 0.286 m.
-      Volume perpindahan air kotak ~0.0340 m^3 -> gaya apung setara ~34.05 kg.
-      Massa total (base + 6 thruster) dibuat SEDIKIT DI BAWAH itu supaya ROV
-      apung pelan saat thruster mati (near-neutral, sedikit positif).
+    * Bbox visual/mounting (body_x/y/z) = 0.345 x 0.345 x 0.286 m, TAPI collision
+      box sumber buoyancy (buoy_x/y/z, dari rov_params.yaml: buoyancy_collision)
+      diskalakan LEBIH KECIL: rangka ROV asli berongga, volume perpindahan air
+      efektif hanya dari kompartemen tersegel, bukan seluruh bbox luar.
+      Massa total (base + 6 thruster + gripper, ~8.7 kg) dibuat SEDIKIT DI BAWAH
+      massa air yg dipindahkan collision box itu supaya ROV apung pelan saat
+      thruster mati (near-neutral, sedikit positif).
       Ini placeholder yang di-tune di M2, BUKAN massa ROV asli.
     * Koefisien hidrodinamika memakai nilai acuan tipe BlueROV2 (di-tune belakangan).
@@ -35,4 +38,7 @@
   <xacro:property name="thruster_mass" value="${rp['thruster_mass']}"/>
   <xacro:property name="fluid_density" value="${rp['fluid_density']}"/>
+  <xacro:property name="buoy_x" value="${rp['buoyancy_collision']['x']}"/>
+  <xacro:property name="buoy_y" value="${rp['buoyancy_collision']['y']}"/>
+  <xacro:property name="buoy_z" value="${rp['buoyancy_collision']['z']}"/>
   <xacro:property name="cog" value="${rp['cog']}"/>
   <!-- Tensor inertia base_link (kg*m^2) di CoG — dari YAML (dihitung oleh
@@ -103,4 +109,7 @@
     </visual>
     <!-- Collision box dipakai plugin Buoyancy untuk menghitung volume perpindahan.
+         Ukuran (buoy_x/y/z) SENGAJA lebih kecil dari bbox visual/mounting body_x/y/z
+         (rangka ROV asli berongga, volume perpindahan efektif hanya dari
+         kompartemen tersegel); lihat rov_params.yaml: buoyancy_collision.
          Origin digeser ke atas sebesar cob.z (relatif thd inertial origin/CoG di atas)
          agar CoB (centroid box ini) berada di atas CoG -> metacentric height positif,
@@ -109,5 +118,5 @@
       <origin xyz="${rp['cob']['x']} ${rp['cob']['y']} ${rp['cob']['z']}" rpy="0 0 0"/>
       <geometry>
-        <box size="${body_x} ${body_y} ${body_z}"/>
+        <box size="${buoy_x} ${buoy_y} ${buoy_z}"/>
       </geometry>
     </collision>
